File: KiCad_Files/NodeStandard/NodeStandard.sch (KiCad schematic (older format))
At the start: 107 parts, among them J1 AC Current In, J10 Opto Coupler 1 in, J11 Opto Coupler 2 in, J12 Opto Coupler 3 in, J13 Relay 1 Output, J14 Relay 2 Output, J15 Switch 3 in, J16 Switch 2 in, J17 Switch 1 in, J18 Force output FET 1 on, J19 Force output FET 2 on, J2 Current coil in, J20 FET 1 Output, J21 FET 2 Output, J22 Force output Relay 3 on, J23 Relay 3 Output 1, J24 Relay 3 Output 2, J25 230VAC in, J26 5V-in, J27 ExtDC-in, J28 Hal current sensor, J29 Current sensor select, J3 AC Current loop, J4 EXT1, J5 OledDisplay, J6 RFIDReader, J7 EXT2, J8 Force output Relay 1 on, J9 Force output Relay 2 on, K1 SANYOU_SRD_Form_C, K2 SANYOU_SRD_Form_C, K3 RT42xAxx, Q1 BC547, Q2 BC547, Q3 IRLZ34N, Q4 IRLZ34N, Q5 BC547, U1 MCP23017_SP

Commit message: V0.0.9.0 added a number of improvements
Parts:
- added LM2596IN+1: IN+, TestPoint:TestPoint_THTPad_2.0x2.0mm_Drill1.0mm, symbol Connector:TestPoint
- added LM2596IN-1: IN-, TestPoint:TestPoint_THTPad_2.0x2.0mm_Drill1.0mm, symbol Connector:TestPoint
- added LM2596Out+1: Out+, TestPoint:TestPoint_THTPad_2.0x2.0mm_Drill1.0mm, symbol Connector:TestPoint
- added LM2596Out-1: OUT-, TestPoint:TestPoint_THTPad_2.0x2.0mm_Drill1.0mm, symbol Connector:TestPoint
- added Q6: 2N3906, Package_TO_SOT_THT:TO-92_Inline, symbol Transistor_BJT:2N3906
- added R30: 1k, Resistor_THT:R_Axial_DIN0207_L6.3mm_D2.5mm_P7.62mm_Horizontal, symbol Device:R
- added TP5: La, TestPoint:TestPoint_THTPad_2.0x2.0mm_Drill1.0mm, symbol Connector:TestPoint
- added TP6: Lb, TestPoint:TestPoint_THTPad_2.0x2.0mm_Drill1.0mm, symbol Connector:TestPoint
- J25: value 230VAC in -> 230VAC/12-40VDC in
Connections:
- net +3V3: now also Q6.1 (E); no longer J5.3 (Pin_3), J6.3 (Pin_3), R2.1, R4.1
- net +5V: now also LM2596Out+1.1
- net 230VAC-L: now also LM2596IN+1.1
- net 230VAC-N: now also LM2596IN-1.1
- net GND: now also LM2596Out-1.1
- net GPIO15_HS2_CMD: now also R30.1
- net at J2.TN, L1.1, R1.2: now also TP5.1
- net at J2.S, L1.2, R1.1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: now also TP6.1
- new net: J5.3 (Pin_3), J6.3 (Pin_3), Q6.3 (C), R2.1, R4.1
- new net: Q6.2 (B), R30.2
- no-connect marks 23 -> 22
Changed lines of the file:
@@
 Sheet 1 1
 Title "Node Standard"
-Date "2021-02-20"
+Date "2021-04-23"
 Rev "V0.9"
 Comp "MakerSpace Leiden"
@@
 P 15425 2300
 F 0 "J25" H 15375 2450 50  0000 L CNN
-F 1 "230VAC in" H 15575 2450 50  0000 L CNN
+F 1 "230VAC/12-40VDC in" H 15050 2100 50  0000 L CNN
 F 2 "Connector_Phoenix_MSTB:PhoenixContact_MSTB_2,5_2-GF-5,08_1x02_P5.08mm_Horizontal_ThreadedFlange" H 15425 2300 50  0001 C CNN
 F 3 "~" H 15425 2300 50  0001 C CNN
@@
 L power:+3.3V #PWR09
 U 1 1 5FF4729E
-P 3625 3025
-F 0 "#PWR09" H 3625 2875 50  0001 C CNN
-F 1 "+3.3V" V 3640 3153 50  0000 L CNN
-F 2 "" H 3625 3025 50  0001 C CNN
-F 3 "" H 3625 3025 50  0001 C CNN
-	1    3625 3025
-	0    1    -1   0
+P 4775 2300
+F 0 "#PWR09" H 4775 2150 50  0001 C CNN
+F 1 "+3.3V" V 4790 2428 50  0000 L CNN
+F 2 "" H 4775 2300 50  0001 C CNN
+F 3 "" H 4775 2300 50  0001 C CNN
+	1    4775 2300
+	-1   0    0    -1
 $EndComp
-Wire Wire Line
-	3625 3025 3025 3025
 Text GLabel 1875 7825 0    50   BiDi ~ 0
 GPIO13_I2C-SDA
@@
 Wire Wire Line
 	3025 2425 3200 2425
-Connection ~ 3025 3025
 Wire Wire Line
 	3025 3025 2775 3025
@@
 Wire Wire Line
 	2775 4025 3700 4025
-$Comp
-L power:+3.3V #PWR010
-U 1 1 5FB1C92F
-P 3625 3925
-F 0 "#PWR010" H 3625 3775 50  0001 C CNN
-F 1 "+3.3V" V 3640 4053 50  0000 L CNN
-F 2 "" H 3625 3925 50  0001 C CNN
-F 3 "" H 3625 3925 50  0001 C CNN
-	1    3625 3925
-	0    1    -1   0
-$EndComp
 Wire Wire Line
 	2775 3725 3350 3725
 Wire Wire Line
-	2775 3925 3625 3925
+	2775 3925 3025 3925
 Wire Wire Line
 	2775 3825 3350 3825
@@
 	1950 6000 1950 6350
 Wire Wire Line
-	1950 6350 2325 6350
+	1950 6350 2125 6350
 Wire Wire Line
 	1950 5600 2950 5600
@@
 Text GLabel 4500 1200 2    50   Input ~ 0
 GPI34_BUT1
-Text GLabel 4500 1300 2    50   BiDi ~ 0
+Text GLabel 4900 3175 2    50   BiDi ~ 0
 GPIO15_HS2_CMD
 Text GLabel 4500 1400 2    50   BiDi ~ 0
@@
 NoConn ~ 1325 1675
 NoConn ~ 4500 1200
-NoConn ~ 4500 1300
 NoConn ~ 3400 8325
 NoConn ~ 3400 8425
@@
 	2375 5200 2375 4850
 Connection ~ 2950 5200
+$Comp
+L Transistor_BJT:2N3906 Q6
+U 1 1 60828342
+P 4575 2525
+F 0 "Q6" V 4903 2525 50  0000 C CNN
+F 1 "2N3906" V 4812 2525 50  0000 C CNN
+F 2 "Package_TO_SOT_THT:TO-92_Inline" H 4775 2450 50  0001 L CIN
+F 3 "https://www.onsemi.com/pub/Collateral/2N3906-D.PDF" H 4575 2525 50  0001 L CNN
+	1    4575 2525
+	0    -1   -1   0
+$EndComp
+$Comp
+L Device:R R30
+U 1 1 608BD903
+P 4575 2950
+F 0 "R30" V 4475 2900 50  0000 L CNN
+F 1 "1k" V 4575 2900 50  0000 L CNN
+F 2 "Resistor_THT:R_Axial_DIN0207_L6.3mm_D2.5mm_P7.62mm_Horizontal" V 4505 2950 50  0001 C CNN
+F 3 "~" H 4575 2950 50  0001 C CNN
+	1    4575 2950
+	-1   0    0    1
+$EndComp
+Wire Wire Line
+	4575 2800 4575 2725
+Wire Wire Line
+	4575 3100 4575 3175
+Wire Wire Line
+	4575 3175 4900 3175
+Wire Wire Line
+	4775 2300 4775 2425
+Wire Wire Line
+	3200 2425 4375 2425
+Connection ~ 3200 2425
+Connection ~ 3025 3025
+$Comp
+L power:GND #PWR0101
+U 1 1 60A7507A
+P 13600 5300
+F 0 "#PWR0101" H 13600 5050 50  0001 C CNN
+F 1 "GND" H 13605 5127 50  0000 C CNN
+F 2 "" H 13600 5300 50  0001 C CNN
+F 3 "" H 13600 5300 50  0001 C CNN
+	1    13600 5300
+	1    0    0    -1
+$EndComp
+$Comp
+L power:+5V #PWR0102
+U 1 1 60A7587B
+P 13600 4800
+F 0 "#PWR0102" H 13600 4650 50  0001 C CNN
+F 1 "+5V" H 13615 4973 50  0000 C CNN
+F 2 "" H 13600 4800 50  0001 C CNN
+F 3 "" H 13600 4800 50  0001 C CNN
+	1    13600 4800
+	1    0    0    -1
+$EndComp
+Wire Wire Line
+	13600 4800 13600 4925
+Wire Wire Line
+	13600 4925 13775 4925
+Wire Wire Line
+	13600 5300 13600 5225
+Wire Wire Line
+	13600 5225 13775 5225
+Text GLabel 14950 5225 2    50   Output ~ 0
+230VAC-N
+Text GLabel 14950 4925 2    50   Output ~ 0
+230VAC-L
+Wire Wire Line
+	14600 4925 14950 4925
+Wire Wire Line
+	14950 5225 14600 5225
+$Comp
+L Connector:TestPoint LM2596IN+1
+U 1 1 6086A970
+P 14600 4925
+F 0 "LM2596IN+1" H 14658 5043 50  0000 L CNN
+F 1 "IN+" H 14658 4952 50  0000 L CNN
+F 2 "TestPoint:TestPoint_THTPad_2.0x2.0mm_Drill1.0mm" H 14800 4925 50  0001 C CNN
+F 3 "~" H 14800 4925 50  0001 C CNN
+	1    14600 4925
+	1    0    0    -1
+$EndComp
+$Comp
+L Connector:TestPoint LM2596Out+1
+U 1 1 60871FAC
+P 13775 4925
+F 0 "LM2596Out+1" H 13833 5043 50  0000 L CNN
+F 1 "Out+" H 13833 4952 50  0000 L CNN
+F 2 "TestPoint:TestPoint_THTPad_2.0x2.0mm_Drill1.0mm" H 13975 4925 50  0001 C CNN
+F 3 "~" H 13975 4925 50  0001 C CNN
+	1    13775 4925
+	1    0    0    -1
+$EndComp
+$Comp
+L Connector:TestPoint LM2596IN-1
+U 1 1 60872707
+P 14600 5225
+F 0 "LM2596IN-1" H 14658 5343 50  0000 L CNN
+F 1 "IN-" H 14658 5252 50  0000 L CNN
+F 2 "TestPoint:TestPoint_THTPad_2.0x2.0mm_Drill1.0mm" H 14800 5225 50  0001 C CNN
+F 3 "~" H 14800 5225 50  0001 C CNN
+	1    14600 5225
+	1    0    0    -1
+$EndComp
+$Comp
+L Connector:TestPoint LM2596Out-1
+U 1 1 608BEFE4
+P 13775 5225
+F 0 "LM2596Out-1" H 13833 5343 50  0000 L CNN
+F 1 "OUT-" H 13833 5252 50  0000 L CNN
+F 2 "TestPoint:TestPoint_THTPad_2.0x2.0mm_Drill1.0mm" H 13975 5225 50  0001 C CNN
+F 3 "~" H 13975 5225 50  0001 C CNN
+	1    13775 5225
+	1    0    0    -1
+$EndComp
+$Comp
+L Connector:TestPoint TP5
+U 1 1 60811CBC
+P 2125 6300
+F 0 "TP5" H 2183 6418 50  0000 L CNN
+F 1 "La" H 2183 6327 50  0000 L CNN
+F 2 "TestPoint:TestPoint_THTPad_2.0x2.0mm_Drill1.0mm" H 2325 6300 50  0001 C CNN
+F 3 "~" H 2325 6300 50  0001 C CNN
+	1    2125 6300
+	1    0    0    -1
+$EndComp
+Wire Wire Line
+	2125 6300 2125 6350
+Connection ~ 2125 6350
+Wire Wire Line
+	2125 6350 2325 6350
+$Comp
+L Connector:TestPoint TP6
+U 1 1 608599A5
+P 3075 6300
+F 0 "TP6" H 3133 6418 50  0000 L CNN
+F 1 "Lb" H 3133 6327 50  0000 L CNN
+F 2 "TestPoint:TestPoint_THTPad_2.0x2.0mm_Drill1.0mm" H 3275 6300 50  0001 C CNN
+F 3 "~" H 3275 6300 50  0001 C CNN
+	1    3075 6300
+	1    0    0    -1
+$EndComp
+Wire Wire Line
+	2950 6350 3075 6350
+Wire Wire Line
+	3075 6350 3075 6300
+Connection ~ 2950 6350
+Wire Wire Line
+	3025 3025 3025 3925
 $EndSCHEMATC
